Commit message: fix&feat: [olga_hand/urdf]: Fix joint axis of second finger & add box collision

File: Hand Olga/urdf/hand_asembly_ver2_URDF_5.urdf (robot description, URDF)
Before this commit: robot hand_asembly_ver2_URDF_5, 10 links, 9 joints
Links:
- link base_link: geometry collision box size=0.13 0.08 0.056; visual mesh filename=base_link.STL
- link distal_finger_first: geometry collision box size=0.04 0.03 0.04; visual mesh filename=distal_finger_first.STL
- link distal_finger_second: geometry collision box size=0.04 0.03 0.04; visual mesh filename=distal_finger_second.STL
- link distal_thumb: geometry collision box size=0.04 0.03 0.04; visual mesh filename=distal_thumb.STL
- link mideal_finger_first: geometry collision box size=0.04 0.03 0.04; visual mesh filename=mideal_finger_first.STL
- link mideal_finger_second: geometry collision box size=0.04 0.03 0.04; visual mesh filename=mideal_finger_second.STL
- link mideal_thumb: geometry collision box size=0.04 0.03 0.05; visual mesh filename=mideal_thumb.STL
- link proximal_finger_first: geometry visual mesh filename=proximal_finger_first.STL
- link proximal_finger_second: geometry visual mesh filename=proximal_finger_second.STL
- link proximal_thumb: geometry visual mesh filename=proximal_thumb.STL
Joints:
- joint joint_distal_finger_first: limit lower=-1.57 upper=1.57 effort=0 velocity=0 -> lower=-1.57 upper=1.57 effort=0.35 velocity=1.
- joint joint_distal_finger_second: axis -1 0 0 -> 1 0 0; limit lower=0 upper=0 effort=0 velocity=0 -> lower=-1.57 upper=1.57 effort=0.35 velocity=1.
- joint joint_distal_thumb: limit lower=-1.57 upper=1.57 effort=0 velocity=0 -> lower=-1.57 upper=1.57 effort=0.35 velocity=1.
- joint joint_mideal_finger_first: limit lower=0 upper=1.0 effort=0 velocity=0 -> lower=0 upper=1.0 effort=0.35 velocity=1.
- joint joint_mideal_finger_second: axis -1 0 0 -> 1 0 0; limit lower=0 upper=0 effort=0 velocity=0 -> lower=0 upper=1.0 effort=0.35 velocity=1
- joint joint_mideal_thumb: limit lower=0 upper=1.0 effort=0 velocity=0 -> lower=0 upper=1.0 effort=0.35 velocity=1.
- joint joint_proximal_thumb: limit lower=-3.14 upper=0 effort=0 velocity=0 -> lower=-3.14 upper=0 effort=0.35 velocity=1.
